Commit message: resolving urdf issues

File: titan_description/urdf/corrected_titan.urdf (robot description, URDF)
Before this commit: robot TITAN_V2_TURTLEBOT_FINAL_ASSLY_UPDATED (1).SLDASM, 8 links, 7 joints
Links:
- link Depth_Camera_Link: geometry collision mesh filename=package://corrected titan urdf/meshes/Depth_Camera_Link.STL; visual mesh filename=package://corrected titan urdf/meshes/Depth_Camera_Link.STL
- link Front_Caster_Link: geometry collision mesh filename=package://corrected titan urdf/meshes/Front_Caster_Link.STL; visual mesh filename=package://corrected titan urdf/meshes/Front_Caster_Link.STL
- link Left_Wheel_Link: mass 0.0351745701969681 -> 0.03517457019697; geometry collision mesh filename=package://corrected titan urdf/meshes/Left_Wheel_Link.STL; visual mesh filename=package://corrected titan urdf/meshes/Left_Wheel_Link.STL
- link Lidar_Link: geometry collision mesh filename=package://corrected titan urdf/meshes/Lidar_Link.STL; visual mesh filename=package://corrected titan urdf/meshes/Lidar_Link.STL
- link Rear_Caster_Link: geometry collision mesh filename=package://corrected titan urdf/meshes/Rear_Caster_Link.STL; visual mesh filename=package://corrected titan urdf/meshes/Rear_Caster_Link.STL
- link Right_Wheel_Link: mass 0.0351745248993485 -> 0.0351745248993403; geometry collision mesh filename=package://corrected titan urdf/meshes/Right_Wheel_Link.STL; visual mesh filename=package://corrected titan urdf/meshes/Right_Wheel_Link.STL
- link base_link: mass 0.920547254934808 -> 0.9205472549348; geometry collision mesh filename=package://corrected titan urdf/meshes/base_link.STL; visual mesh filename=package://corrected titan urdf/meshes/base_link.STL
- link camera_link: geometry collision mesh filename=package://corrected titan urdf/meshes/camera_link.STL; visual mesh filename=package://corrected titan urdf/meshes/camera_link.STL
Joints:
- joint Depth_Camera_Joint: origin xyz=0.063825 -0.00022394 0.20111 rpy=0 0 0 -> xyz=0.06382528434402 -0.000223937751711724 0.20110747354824 rpy=0 0 0
- joint Front_Caster_Joint: origin xyz=0.099797 0 -0.005 rpy=0 0 0 -> xyz=0.0997970587698719 0 -0.0050000002459 rpy=0 0 0
- joint Left_Wheel_Joint: axis 0 1 0 -> 0 -1 0; origin xyz=0.0001 0.09075 0.022 rpy=0 0 3.1416 -> xyz=9.9999806285E-05 0.09075 0.022 rpy=0 0 0
- joint Lidar_Joint: origin xyz=0.065 0 0.15166 rpy=0 0 0 -> xyz=0.065 0 0.15165774394 rpy=0 0 0; type fixed -> continuous
- joint Rear_Caster_Joint: origin xyz=-0.1 0.00020294 -0.005 rpy=0 0 0 -> xyz=-0.1 0.000202941230128117 -0.0050000002459 rpy=0 0 0
- joint Right_Wheel_Joint: axis 0 1 0 -> 0 -0.999999999990373 0; origin xyz=0.0001 -0.0905 0.022 rpy=0 0 3.1416 -> xyz=9.9999806285E-05 -0.090499999999896 0.022 rpy=0 0 0
- joint camera_joint: origin xyz=0.13025 0 0.088971 rpy=0 0 0 -> xyz=0.130254250725601 0 0.0889713517135 rpy=0 0 0
