Commit message: some change in trail.urdf

File: titan_description/urdf/trial.urdf (robot description, URDF)
Before this commit: robot titan, 9 links, 8 joints
Links:
- link Depth_Camera_Link: geometry collision mesh filename=package://titan_description/meshes/tmesh/Depth_Camera_Link.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; visual mesh filename=package://titan_description/meshes/tmesh/Depth_Camera_Link.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
- link Front_Caster_Link: geometry collision mesh filename=package://titan_description/meshes/tmesh/Front_Caster_Link.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; visual mesh filename=package://titan_description/meshes/tmesh/Front_Caster_Link.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
- link Lidar_Link: geometry collision mesh filename=package://titan_description/meshes/tmesh/Lidar_Link.STL; visual mesh filename=package://titan_description/meshes/tmesh/Lidar_Link.STL
- link Rear_Caster_Link: geometry collision mesh filename=package://titan_description/meshes/tmesh/Rear_Caster_Link.S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; visual mesh filename=package://titan_description/meshes/tmesh/Rear_Caster_Link.S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
- link base_link: geometry collision mesh filename=package://titan_description/meshes/tmesh/base_link.STL; visual mesh filename=package://titan_description/meshes/tmesh/base_link.STL
Joints:
- joint Depth_Camera_Joint: origin xyz=-0.063825 0.00022394 0.20111 rpy=0 0 3.14159265 -> xyz=-0.063825 0.00022394 0.20111 rpy=0 0 0
- joint Front_Caster_Joint: origin xyz=-0.099797 0 -0.005 rpy=0 0 3.14159265 -> xyz=-0.099797 0 -0.005 rpy=0 0 0
- joint Left_Wheel_Joint: origin xyz=-0.0001 -0.09075 0.022 rpy=0 0 3.14159265 -> xyz=-0.0001 -0.09075 0.022 rpy=0 0 0
- joint Lidar_Joint: origin xyz=-0.065 0 0.15166 rpy=0 0 3.14159265 -> xyz=-0.065 0 0.15166 rpy=0 0 0
- joint RGB_Camera_Joint: origin xyz=-0.13025 0 0.088971 rpy=0 0 3.14159265 -> xyz=-0.13025 0 0.088971 rpy=0 0 0
- joint Rear_Caster_Joint: origin xyz=0.1 -0.00020294 -0.005 rpy=0 0 3.14159265 -> xyz=0.1 -0.00020294 -0.005 rpy=0 0 0
- joint Right_Wheel_Joint: origin xyz=-0.0001 0.0905 0.022 rpy=0 0 3.14159265 -> xyz=-0.0001 0.0905 0.022 rpy=0 0 0
- joint base_link_joint: origin xyz=0 0 0 rpy=0 0 3.14159265 -> xyz=0 0 0 rpy=0 0 0
