Commit message: setting up usbs and correcting laserscan

File: titan_description/urdf/turtlebot3_burger.urdf (robot description, URDF)
Before this commit: robot turtlebot3_burger, 7 links, 6 joints
Links:
- removed link ${namespace}base_scan
- added link ${namespace}laser, mass 0.114; collision cylinder length=0.0315 radius=0.055; visual mesh filename=package://turtlebot3_description/meshes/sensors/lds.stl scale=0.001 0.001 0.001
Joints:
- joint ${namespace}scan_joint: child ${namespace}base_scan -> ${namespace}laser

Commit message: office maps

File: titan_description/urdf/turtlebot3_burger.urdf (robot description, URDF)
Before this commit: robot turtlebot3_burger, 7 links, 6 joints
Joints:
- joint ${namespace}scan_joint: origin xyz=-0.032 0 0.172 rpy=0 0 0 -> xyz=-0.072 0 0.172 rpy=0 0 0

Commit message: bringup and shell script changes

File: titan_description/urdf/turtlebot3_burger.urdf (robot description, URDF)
Before this commit: robot turtlebot3_burger, 7 links, 6 joints
Joints:
- joint ${namespace}scan_joint: origin xyz=-0.072 0 0.172 rpy=0 0 0 -> xyz=-0.072 0 0.172 rpy=0 0 3.14159

Commit message: deleted unwanted files and comments

File: titan_description/urdf/turtlebot3_burger.urdf (robot description, URDF)
Before this commit: robot turtlebot3_burger, 7 links, 6 joints
Joints:
- joint ${namespace}scan_joint: origin xyz=-0.072 0 0.172 rpy=0 0 3.14159 -> xyz=-0.072 0 0.172 rpy=0 0 0

Commit message: rotated urdf joints by 180

File: titan_description/urdf/turtlebot3_burger.urdf (robot description, URDF)
Before this commit: robot turtlebot3_burger, 7 links, 6 joints
Links:
- removed link ${namespace}imu_link
Joints:
- removed joint ${namespace}imu_joint
- joint ${namespace}caster_back_joint: origin xyz=-0.081 0 -0.004 rpy=-1.57 0 0 -> xyz=-0.081 0 -0.004 rpy=-1.57 0 3.1416
- joint ${namespace}scan_joint: origin xyz=-0.072 0 0.172 rpy=0 0 0 -> xyz=0.072 0 0.172 rpy=0 0 0
- joint ${namespace}wheel_left_joint: origin xyz=0.0 0.08 0.023 rpy=-1.57 0 0 -> xyz=0.0 0.08 0.023 rpy=-1.57 0 3.1416
- joint ${namespace}wheel_right_joint: origin xyz=0.0 -0.080 0.023 rpy=-1.57 0 0 -> xyz=0.0 -0.080 0.023 rpy=-1.57 0 3.1416

Commit message: wheel joints converted to fixed joints

File: titan_description/urdf/turtlebot3_burger.urdf (robot description, URDF)
Before this commit: robot turtlebot3_burger, 6 links, 5 joints
Joints:
- joint ${namespace}wheel_left_joint: axis 0 0 1 -> (none); type continuous -> fixed
- joint ${namespace}wheel_right_joint: axis 0 0 1 -> (none); type continuous -> fixed

Commit message: copied files from v2

File: titan_description/urdf/turtlebot3_burger.urdf (robot description, URDF)
Before this commit: robot turtlebot3_burger, 7 links, 6 joints
Links:
- removed link ${namespace}imu_link
Joints:
- removed joint ${namespace}imu_joint
- joint ${namespace}caster_back_joint: origin xyz=-0.081 0 -0.004 rpy=-1.57 0 0 -> xyz=-0.081 0 -0.004 rpy=-1.57 0 3.1416
- joint ${namespace}scan_joint: origin xyz=-0.072 0 0.172 rpy=0 0 0 -> xyz=0.072 0 0.172 rpy=0 0 0
- joint ${namespace}wheel_left_joint: axis 0 0 1 -> (none); origin xyz=0.0 0.08 0.023 rpy=-1.57 0 0 -> xyz=0.0 0.08 0.023 rpy=-1.57 0 3.1416; type continuous -> fixed
- joint ${namespace}wheel_right_joint: axis 0 0 1 -> (none); origin xyz=0.0 -0.080 0.023 rpy=-1.57 0 0 -> xyz=0.0 -0.080 0.023 rpy=-1.57 0 3.1416; type continuous -> fixed

Commit message: modify shell script

File: titan_description/urdf/turtlebot3_burger.urdf (robot description, URDF)
Before this commit: robot turtlebot3_burger, 6 links, 5 joints
Joints:
- joint ${namespace}scan_joint: origin xyz=0.072 0 0.172 rpy=0 0 0 -> xyz=0.072 0 0.172 rpy=0 0 3.14159

Commit message: urdf resolved and submodules added for this branch

File: titan_description/urdf/turtlebot3_burger.urdf (robot description, URDF)
Before this commit: robot turtlebot3_burger, 7 links, 6 joints
Links:
- removed link ${namespace}imu_link
Joints:
- removed joint ${namespace}imu_joint
- joint ${namespace}caster_back_joint: origin xyz=-0.081 0 -0.004 rpy=-1.57 0 0 -> xyz=-0.081 0 -0.004 rpy=-1.57 0 3.1416
- joint ${namespace}scan_joint: origin xyz=-0.072 0 0.172 rpy=0 0 0 -> xyz=0.072 0 0.172 rpy=0 0 3.14159
- joint ${namespace}wheel_left_joint: axis 0 0 1 -> (none); origin xyz=0.0 0.08 0.023 rpy=-1.57 0 0 -> xyz=0.0 0.08 0.023 rpy=-1.57 0 3.1416; type continuous -> fixed
- joint ${namespace}wheel_right_joint: axis 0 0 1 -> (none); origin xyz=0.0 -0.080 0.023 rpy=-1.57 0 0 -> xyz=0.0 -0.080 0.023 rpy=-1.57 0 3.1416; type continuous -> fixed
