Commit message: solve urdf and scan topic issue

File: titan_description/urdf/titan.urdf (robot description, URDF)
Before this commit: robot titan, 9 links, 8 joints
Links:
- removed link Lidar_Link
- added link laser, mass 0.16538; collision mesh filename=package://titan_description/meshes/titan_meshes/Lidar_Link.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; visual mesh filename=package://titan_description/meshes/titan_meshes/Lidar_Link.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
Joints:
- removed joint Lidar_Joint
- added joint scan_joint: type fixed, parent base_link, child laser, origin xyz=-0.065 0 0.15166 rpy=0 0 3.14159265, axis 0 0 1, limit effort=0.1 velocity=65

Commit message: solving lidar issue

File: titan_description/urdf/titan.urdf (robot description, URDF)
Before this commit: robot titan, 9 links, 8 joints
Links:
- removed link laser
- added link Lidar_Link, mass 0.16538; collision mesh filename=package://titan_description/meshes/titan_meshes/Lidar_Link.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; visual mesh filename=package://titan_description/meshes/titan_meshes/Lidar_Link.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
Joints:
- removed joint scan_joint
- added joint Lidar_Joint: type fixed, parent base_link, child Lidar_Link, origin xyz=-0.065 0 0.15166 rpy=0 0 3.14159265, axis 0 0 1, limit effort=0.1 velocity=65

Commit message: slam issue resolved, turned lidar link transform by 180 degrees

File: titan_description/urdf/titan.urdf (robot description, URDF)
Before this commit: robot titan, 9 links, 8 joints
Joints:
- joint Lidar_Joint: origin xyz=-0.065 0 0.15166 rpy=0 0 3.14159265 -> xyz=-0.065 0 0.15166 rpy=0 0 0

Commit message: resolving transform issues

File: titan_description/urdf/titan.urdf (robot description, URDF)
Before this commit: robot titan, 9 links, 8 joints
Joints:
- joint Depth_Camera_Joint: origin xyz=-0.063825 0.00022394 0.20111 rpy=0 0 3.14159265 -> xyz=-0.063825 0.00022394 0.20111 rpy=0 0 0
- joint Front_Caster_Joint: origin xyz=-0.099797 0 -0.005 rpy=0 0 3.14159265 -> xyz=-0.099797 0 -0.005 rpy=0 0 0
- joint Left_Wheel_Joint: origin xyz=-0.0001 -0.09075 0.022 rpy=0 0 3.14159265 -> xyz=-0.0001 -0.09075 0.022 rpy=0 0 0
- joint RGB_Camera_Joint: origin xyz=-0.13025 0 0.088971 rpy=0 0 3.14159265 -> xyz=-0.13025 0 0.088971 rpy=0 0 0
- joint Rear_Caster_Joint: origin xyz=0.1 -0.00020294 -0.005 rpy=0 0 3.14159265 -> xyz=0.1 -0.00020294 -0.005 rpy=0 0 0
- joint Right_Wheel_Joint: origin xyz=-0.0001 0.0905 0.022 rpy=0 0 3.14159265 -> xyz=-0.0001 0.0905 0.022 rpy=0 0 0
- joint base_link_joint: origin xyz=0 0 0 rpy=0 0 3.14159265 -> xyz=0 0 0 rpy=0 0 0

Commit message: edit new urdf file

File: titan_description/urdf/titan.urdf (robot description, URDF)
Before this commit: robot titan, 9 links, 8 joints
Links:
- removed link Depth_Camera_Link
- removed link Front_Caster_Link
- removed link Lidar_Link
- removed link RGB_Camera_Link
- removed link Rear_Caster_Link
Joints:
- removed joint Depth_Camera_Joint
- removed joint Front_Caster_Joint
- removed joint Lidar_Joint
- removed joint RGB_Camera_Joint
- removed joint Rear_Caster_Joint
- joint Left_Wheel_Joint: origin xyz=-0.0001 -0.09075 0.022 rpy=0 0 0 -> xyz=-0.0001 -0.09075 0.022 rpy=0 0 3.14159265
- joint Right_Wheel_Joint: origin xyz=-0.0001 0.0905 0.022 rpy=0 0 0 -> xyz=-0.0001 0.0905 0.022 rpy=0 0 3.14159265
- joint base_link_joint: origin xyz=0 0 0 rpy=0 0 0 -> xyz=0 0 0 rpy=0 0 3.14159265

Commit message: resolving urdf issues

File: titan_description/urdf/titan.urdf (robot description, URDF)
Before this commit: robot titan, 4 links, 3 joints
Links:
- added link Depth_Camera_Link, mass 0.081395; collision mesh filename=package://titan_description/meshes/titan_meshes/Depth_Camer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; visual mesh filename=package://titan_description/meshes/titan_meshes/Depth_Camer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
- added link Front_Caster_Link, mass 0.0024002; collision mesh filename=package://titan_description/meshes/titan_meshes/Front_Caste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; visual mesh filename=package://titan_description/meshes/titan_meshes/Front_Caste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
- added link Lidar_Link, mass 0.16538; collision mesh filename=package://titan_description/meshes/titan_meshes/Lidar_Link.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; visual mesh filename=package://titan_description/meshes/titan_meshes/Lidar_Link.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
- added link RGB_Camera_Link, mass 0.01352; collision box size=0.01 0.01 0.01; visual box size=0.01 0.01 0.01
- added link Rear_Caster_Link, mass 0.0024002; collision mesh filename=package://titan_description/meshes/titan_meshes/Rear_Caster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; visual mesh filename=package://titan_description/meshes/titan_meshes/Rear_Caster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
Joints:
- added joint Depth_Camera_Joint: type fixed, parent base_link, child Depth_Camera_Link, origin xyz=-0.063825 0.00022394 0.20111 rpy=0 0 3.14159265, axis 0 0 0
- added joint Front_Caster_Joint: type fixed, parent base_link, child Front_Caster_Link, origin xyz=-0.099797 0 -0.005 rpy=0 0 3.14159265, axis 0 0 0
- added joint Lidar_Joint: type fixed, parent base_link, child Lidar_Link, origin xyz=-0.065 0 0.15166 rpy=0 0 3.14159265, axis 0 0 1, limit effort=0.1 velocity=65
- added joint RGB_Camera_Joint: type fixed, parent base_link, child RGB_Camera_Link, origin xyz=-0.13025 0 0.088971 rpy=0 0 3.14159265, axis 0 0 0
- added joint Rear_Caster_Joint: type fixed, parent base_link, child Rear_Caster_Link, origin xyz=0.1 -0.00020294 -0.005 rpy=0 0 3.14159265, axis 0 0 0
- joint Left_Wheel_Joint: origin xyz=-0.0001 -0.09075 0.022 rpy=0 0 3.14159265 -> xyz=-0.0001 -0.09075 0.022 rpy=0 0 0
- joint Right_Wheel_Joint: origin xyz=-0.0001 0.0905 0.022 rpy=0 0 3.14159265 -> xyz=-0.0001 0.0905 0.022 rpy=0 0 0
- joint base_link_joint: origin xyz=0 0 0 rpy=0 0 3.14159265 -> xyz=0 0 0 rpy=0 0 0

Commit message: Resolved URDF issues

File: titan_description/urdf/titan.urdf (robot description, URDF)
Before this commit: robot titan, 9 links, 8 joints
Joints:
- joint Depth_Camera_Joint: axis 0 0 0 -> (none); origin xyz=-0.063825 0.00022394 0.20111 rpy=0 0 3.14159265 -> xyz=0.063825 0.00022394 0.20111 rpy=0 0 0
- joint Front_Caster_Joint: axis 0 0 0 -> (none); origin xyz=-0.099797 0 -0.005 rpy=0 0 3.14159265 -> xyz=-0.099797 0 -0.005 rpy=0 0 0
- joint Lidar_Joint: axis 0 0 1 -> (none); limit effort=0.1 velocity=65 -> (none); origin xyz=-0.065 0 0.15166 rpy=0 0 3.14159265 -> xyz=0.065 0 0.15166 rpy=0 0 3.14159265
- joint RGB_Camera_Joint: axis 0 0 0 -> (none); origin xyz=-0.13025 0 0.088971 rpy=0 0 3.14159265 -> xyz=0.13025 0 0.088971 rpy=0 0 0
- joint Rear_Caster_Joint: axis 0 0 0 -> (none); origin xyz=0.1 -0.00020294 -0.005 rpy=0 0 3.14159265 -> xyz=0.1 -0.00020294 -0.005 rpy=0 0 0

Commit message: Fix frame URDF for correct transformation references

File: titan_description/urdf/titan.urdf (robot description, URDF)
Before this commit: robot titan, 9 links, 8 joints
Joints:
- joint base_link_joint: child base_link -> base_footprint; parent base_footprint -> base_link
